Commit message: adding masses to links

File: cob_hardware_config/robots/baker/urdf/baker.urdf.xacro (robot description, xacro)
@@ -7,5 +7,7 @@
   <xacro:include filename="$(find cob_description)/urdf/baker_arm/baker_arm.urdf.xacro" />
   <!-- Used for fixing robot to Gazebo -->
-  <link name="world"/>
+  <link name="world">
+    <origin xyz="0 0 0" rpy="0 0 0"/>
+  </link>
   <xacro:baker name="arm" parent="world">
     <origin xyz="0 0 0" rpy="0 0 0" />

Commit message: Baker robot: added arm and gripper links  without gripper fingers in urdf

File: cob_hardware_config/robots/baker/urdf/baker.urdf.xacro (robot description, xacro)
@@ -7,9 +7,5 @@
   <xacro:include filename="$(find cob_description)/urdf/baker_arm/baker_arm.urdf.xacro" />
   <!-- Used for fixing robot to Gazebo -->
-  <link name="world">
-    <origin xyz="0 0 0" rpy="0 0 0"/>
-  </link>
-  <xacro:baker name="arm" parent="world">
-    <origin xyz="0 0 0" rpy="0 0 0" />
-  </xacro:baker>
+  <link name="world"/>
+  <xacro:baker name="arm" parent="world"/>
 </robot>
