Commit message: Improved P-Rob arm configuration, changed UR10 arm to P-Rob arm in raw3-1 robot, updated moveit configs of p_rob and raw3-1

File: cob_hardware_config/robots/p_rob/urdf/p_rob.urdf.xacro (robot description, xacro)
@@ -1,42 +1,13 @@
 <?xml version="1.0"?>
-<robot xmlns:xacro="http://www.ros.org/wiki/xacro"
-       name="p_rob" >
+<robot xmlns:xacro="http://www.ros.org/wiki/xacro" name="p_rob" >
   <!-- common stuff -->
   <xacro:include filename="$(find cob_description)/urdf/common.xacro" />
   <xacro:include filename="$(find cob_description)/urdf/materials.urdf.xacro" />
-  <xacro:include filename="$(find cob_hardware_config)/robots/raw3-1/urdf/properties.urdf.xacro" />
-  <!-- raw base -->
-  <xacro:include filename="$(find raw_description)/urdf/base_long/base.urdf.xacro" />
-  <!-- raw tower -->
-  <xacro:include filename="$(find raw_description)/urdf/tower_asymetric/tower.urdf.xacro" />
-  <!-- torso -->
-  <xacro:include filename="$(find raw_description)/urdf/torso/torso.urdf.xacro" />
-  <!-- head -->
-  <xacro:include filename="$(find raw_description)/urdf/head/head.urdf.xacro" />
-  <!-- p_rob -->
-  <xacro:include filename="$(find cob_description)/urdf/p_rob/p_rob.urdf.xacro" />
-  <!-- sensors -->
-  <xacro:include filename="$(find cob_description)/urdf/sensors/sick_s300_laser.urdf.xacro"/>
-  <!-- composition of the robot -->
-  <xacro:raw_base name="base"/>
-  <!-- base laser front -->
-  <xacro:sick_s300_laser_v0 name="base_laser_front" parent="base">
-    <origin xyz="${laser_front_x} ${laser_front_y} ${laser_front_z}" rpy="${laser_front_roll} ${laser_front_pitch} ${laser_front_yaw}" />
-  </xacro:sick_s300_laser_v0>
-  <!-- base laser rear -->
-  <xacro:sick_s300_laser_v0 name="base_laser_rear" parent="base">
-    <origin xyz="${laser_rear_x} ${laser_rear_y} ${laser_rear_z}" rpy="${laser_rear_roll} ${laser_rear_pitch} ${laser_rear_yaw}" />
-  </xacro:sick_s300_laser_v0>
-  <xacro:tower_asymetric name="tower" parent="base_link">
-    <origin xyz="${tower_x} ${tower_y} ${tower_z}" rpy="${tower_roll} ${tower_pitch} ${tower_yaw}" />
-  </xacro:tower_asymetric>
-  <xacro:raw_torso name="torso" parent="base_link">
-    <origin xyz="${torso_x} ${torso_y} ${torso_z}" rpy="${torso_roll} ${torso_pitch} ${torso_yaw}" />
-  </xacro:raw_torso>
-  <xacro:raw_head name="head" parent="torso_2_link">
-    <origin xyz="${head_x} ${head_y} ${head_z}" rpy="${head_roll} ${head_pitch} ${head_yaw}" />
-  </xacro:raw_head>
-  <xacro:p_rob name="arm" parent="base_link">
-    <origin xyz="${arm_x} ${arm_y} ${arm_z}" rpy="${arm_roll} ${arm_pitch} ${arm_yaw+20}" />
+  <!-- p_rob_arm -->
+  <xacro:include filename="$(find raw_description)/urdf/p_rob_arm/p_rob.urdf.xacro" />
+  <!-- Used for fixing robot to Gazebo -->
+  <link name="world"/>
+  <xacro:p_rob name="arm" parent="world">
+    <origin xyz="0 0 0" rpy="0 0 0" />
   </xacro:p_rob>
 </robot>

File: cob_hardware_config/robots/raw3-1/urdf/raw3-1.urdf.xacro (robot description, xacro)
@@ -12,10 +12,6 @@
   <!-- torso -->
   <xacro:include filename="$(find raw_description)/urdf/torso/torso_v2.urdf.xacro" />
- />
-  <!-- ur_arm
-  <xacro:include filename="$(find raw_description)/urdf/ur_arm/ur10_arm.urdf.xacro" />
-  -->
-  <!-- p-rob_arm -->
-  <xacro:include filename="$(find raw_description)/urdf/p_rob/p_rob.urdf.xacro" />
+  <!-- p_rob_arm -->
+  <xacro:include filename="$(find raw_description)/urdf/p_rob_arm/p_rob.urdf.xacro" />
   <!-- vacuum gripper -->
   <xacro:include filename="$(find raw_description)/urdf/vacuum_gripper/gripper.urdf.xacro" />

Commit message: Fixed p_rob urdf: added height of mounting profiles

File: cob_hardware_config/robots/p_rob/urdf/p_rob.urdf.xacro (robot description, xacro)
@@ -9,5 +9,5 @@
   <link name="world"/>
   <xacro:p_rob name="arm" parent="world">
-    <origin xyz="0 0 0" rpy="0 0 0" />
+    <origin xyz="0 0 0.031" rpy="0 0 0" />
   </xacro:p_rob>
 </robot>
