Commit message: few fixes to raw3-1 urdf after rebase

File: cob_hardware_config/robots/raw3-1/urdf/raw3-1.urdf.xacro (robot description, xacro)
@@ -13,6 +13,9 @@
   <xacro:include filename="$(find raw_description)/urdf/torso/torso_v2.urdf.xacro" />
  />
-  <!-- ur_arm -->
-  <xacro:include filename="$(find cob_description)/urdf/ur_arm/ur10_arm.urdf.xacro" />
+  <!-- ur_arm
+  <xacro:include filename="$(find raw_description)/urdf/ur_arm/ur10_arm.urdf.xacro" />
+  -->
+  <!-- p-rob_arm -->
+  <xacro:include filename="$(find raw_description)/urdf/p_rob/p_rob.urdf.xacro" />
   <!-- vacuum gripper -->
   <xacro:include filename="$(find raw_description)/urdf/vacuum_gripper/gripper.urdf.xacro" />
@@ -35,9 +38,6 @@
     <origin xyz="${torso_x} ${torso_y} ${torso_z}" rpy="${torso_roll} ${torso_pitch} ${torso_yaw}" />
   </xacro:raw_torso_v2>
-  <xacro:ur10 name="arm" parent="base_link">
+  <xacro:p_rob name="arm" parent="base_link">
     <origin xyz="${arm_x} ${arm_y} ${arm_z}" rpy="${arm_roll} ${arm_pitch} ${arm_yaw}" />
-  </xacro:ur10>
-  <xacro:vacuum_gripper name="gripper" parent="arm_ee_link">
-    <origin xyz="${gripper_x} ${gripper_y} ${gripper_z}" rpy="${gripper_roll} ${gripper_pitch} ${gripper_yaw}" />
-  </xacro:vacuum_gripper>
+  </xacro:p_rob>
 </robot>

Commit message: Adapter raw3-1 moveit config for p_rob

File: cob_hardware_config/robots/raw3-1/urdf/raw3-1.urdf.xacro (robot description, xacro)
@@ -35,5 +35,5 @@
   </xacro:raw_torso_v2>
   <xacro:p_rob name="arm" parent="base_link">
-    <origin xyz="${arm_x} ${arm_y} ${arm_z}" rpy="${arm_roll} ${arm_pitch} ${arm_yaw}" />
+    <origin xyz="${arm_x} ${arm_y} ${arm_z}" rpy="${arm_roll} ${arm_pitch} ${arm_yaw + 20}" />
   </xacro:p_rob>
 </robot>

Commit message: raw3-1 fixed PRob mounting yaw parameter

File: cob_hardware_config/robots/raw3-1/urdf/raw3-1.urdf.xacro (robot description, xacro)
@@ -35,5 +35,5 @@
   </xacro:raw_torso_v2>
   <xacro:p_rob name="arm" parent="base_link">
-    <origin xyz="${arm_x} ${arm_y} ${arm_z}" rpy="${arm_roll} ${arm_pitch} ${arm_yaw + 20}" />
+    <origin xyz="${arm_x} ${arm_y} ${arm_z}" rpy="${arm_roll} ${arm_pitch} ${arm_yaw - 0.349066}" />
   </xacro:p_rob>
 </robot>

Commit message: raw3-1 urdf: corrected PRob arm yaw

File: cob_hardware_config/robots/raw3-1/urdf/raw3-1.urdf.xacro (robot description, xacro)
@@ -35,5 +35,5 @@
   </xacro:raw_torso_v2>
   <xacro:p_rob name="arm" parent="base_link">
-    <origin xyz="${arm_x} ${arm_y} ${arm_z}" rpy="${arm_roll} ${arm_pitch} ${arm_yaw - 0.349066}" />
+    <origin xyz="${arm_x} ${arm_y} ${arm_z}" rpy="${arm_roll} ${arm_pitch} ${arm_yaw - 3.49066}" />
   </xacro:p_rob>
 </robot>
